File: planck-thk.sch (KiCad schematic (older format))
At the start: 123 parts, among them J2 Conn_01x05, J3 Qwiic, J4 Qwiic, J5 Qwiic, J6 JTAG, J7 ISP, J8 Reset, K1 Switch, K10 Switch, K11 Switch, K12 Switch, K13 Switch, K14 Switch, K15 Switch, K16 Switch, K17 Switch, K18 Switch, K19 Switch, K2 Switch, K20 Switch, K21 Switch, K22 Switch, K23 Switch, K24 Switch, K25 Switch, K26 Switch, K27 Switch, K28 Switch, K29 Switch, K3 Switch, K30 Switch, K31 Switch, K32 Switch, K33 Switch, K34 Switch, K35 Switch, K36 Switch, K37 Switch, K38 Switch, K39 Switch, K4 Switch, K40 Switch, K41 Switch, K42 Switch, K43 Switch, K44 Switch, K45 Switch, K46 Switch, K47 Switch, K48 Switch, K49 Switch, K5 Switch, K6 Switch, K7 Switch, K8 Switch, K9 Switch, SW1 SW_DIP_x04, SW2 Rotary_Encoder, SW3 Rotary_Encoder, U1 ATMEGA32A-PU, U2 LD1117S33TR_SOT223, Y1 Crystal

Commit message: fix isp and jtag, usb port, remove gerbers
Parts:
- J6: footprint Socket_Strips:Socket_Strip_Straight_2x05_Pitch2.54mm -> Pin_Headers:Pin_Header_Straight_2x05_Pitch2.54mm
- J7: footprint Socket_Strips:Socket_Strip_Straight_2x03_Pitch2.54mm -> Pin_Headers:Pin_Header_Straight_2x03_Pitch2.54mm
Changed lines of the file:
@@
 LIBS:contrib
 LIBS:valves
-LIBS:planck-tht-cache
+LIBS:planck-thk-cache
 EELAYER 25 0
 EELAYER END
@@
 F 0 "J6" H 5000 1450 50  0000 C CNN
 F 1 "JTAG" H 5000 850 50  0000 C CNN
-F 2 "Socket_Strips:Socket_Strip_Straight_2x05_Pitch2.54mm" H 4950 1150 50  0001 C CNN
+F 2 "Pin_Headers:Pin_Header_Straight_2x05_Pitch2.54mm" H 4950 1150 50  0001 C CNN
 F 3 "" H 4950 1150 50  0001 C CNN
 	1    4950 1150
@@
 F 0 "J7" H 5000 2150 50  0000 C CNN
 F 1 "ISP" H 5000 1750 50  0000 C CNN
-F 2 "Socket_Strips:Socket_Strip_Straight_2x03_Pitch2.54mm" H 4950 1950 50  0001 C CNN
+F 2 "Pin_Headers:Pin_Header_Straight_2x03_Pitch2.54mm" H 4950 1950 50  0001 C CNN
 F 3 "" H 4950 1950 50  0001 C CNN
 	1    4950 1950
@@
 $EndComp
 $Comp
-L GND #PWR?
+L GND #PWR035
 U 1 1 5B96F685
 P 7450 2400
-F 0 "#PWR?" H 7450 2150 50  0001 C CNN
+F 0 "#PWR035" H 7450 2150 50  0001 C CNN
 F 1 "GND" V 7450 2200 50  0000 C CNN
 F 2 "" H 7450 2400 50  0001 C CNN
